File: MCU.kicad_sch (KiCad schematic)
At the start: 61 parts, among them J2 SPI connector, J3 I2C connector, J6 USART2 connector, J7 Debug, SW2 RESET, U2 STM32G473CCTx, Y2 16MHz

Commit message: feat: added vias
Connections:
- net CAN1_LED_RX: now also U2.2 (PC13); no longer U2.4 (PC15)
- net CAN2_LED_RX: now also U2.4 (PC15); no longer U2.8 (PA0)
- net CAN2_LED_TX: now also U2.8 (PA0); no longer U2.9 (PA1)
- net CAN3_LED_RX: now also U2.9 (PA1); no longer U2.2 (PC13)
Changed lines of the file:
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@@
 	)
 	(label "CAN3_LED_RX"
-		(at 60.96 66.04 0)
-		(effects
-			(font
-				(size 1.27 1.27)
-			)
-			(justify left bottom)
+		(at 121.92 50.8 180)
+		(effects
+			(font
+				(size 1.27 1.27)
+			)
+			(justify right bottom)
 		)
 	)
@@
 	)
 	(label "CAN2_LED_TX"
-		(at 121.92 50.8 180)
+		(at 121.92 48.26 180)
 		(effects
 			(font
@@
 	)
 	(label "CAN1_LED_RX"
-		(at 60.96 71.12 0)
+		(at 60.96 66.04 0)
 		(effects
 			(font
@@
 	)
 	(label "CAN2_LED_RX"
-		(at 121.92 48.26 180)
-		(effects
-			(font
-				(size 1.27 1.27)
-			)
-			(justify right bottom)
-		)
-	)
+		(at 60.96 71.12 0)
+		(effects
+			(font
+				(size 1.27 1.27)
+			)
+			(justify left bottom)
+		)
+	)

Commit message: feat: started writing BOM
Parts:
- C10, C12, C13, C14, C15, C16: LCSC Part # (none) -> C14663; MOUSER PN (none) -> 963-MAJCU168BB7104KT
- C11, C9: LCSC Part # (none) -> C1648; MOUSER PN (none) -> 581-06035A200GAT2A
- C20: LCSC Part # (none) -> C19702; MOUSER PN (none) -> 581-KGM15CR51C106KT
- D24, D25, D28, D29, D32, D33, D43, D44, D45, D46, D47, D48, D50, D51: LCSC Part # (none) -> C77807; MOUSER PN (none) -> 750-CPDH3V3UP
- D26, D27, D30, D31, D34, D35: LCSC Part # (none) -> C7420333; MOUSER PN (none) -> 863-SBAT54SLT1G
- D37, D38, D39: LCSC Part # (none) -> C965799; MOUSER PN (none) -> 720-Q65113A7467
- D40, D41, D42, D49: LCSC Part # (none) -> C7496818; MOUSER PN (none) -> 720-Q65113A5260
- J2: LCSC Part # (none) -> C37208
- J3, J6: LCSC Part # (none) -> C124378
- J7: LCSC Part # (none) -> C22074484; MOUSER PN (none) -> 200-FTSH10701LDVKTR
- R1, R15, R2, R23, R24, R5, R6, R7: LCSC Part # (none) -> C23182; MOUSER PN (none) -> 603-TR0603KR-0747RL
- R10, R11, R12, R13, R14, R22, R9: LCSC Part # (none) -> C23228; MOUSER PN (none) -> 667-ERA-3APB681V
- R16: LCSC Part # (none) -> C25804; MOUSER PN (none) -> 594-MCT06030D1002BPW
- R3, R4: LCSC Part # (none) -> C99782; MOUSER PN (none) -> 603-AR0603JR-074K7L
- SW2: MOUSER PN (none) -> 506-FSMSM
- U2: MOUSER PN (none) -> 511-STM32G473CCT3
- Y2: LCSC Part # (none) -> C6190540; MOUSER PN (none) -> 520-160-18-33-AENTR3

Commit message: feat: finished BOM
Parts:
- D37, D38, D39: MOUSER PN 720-Q65113A7467 -> 604-APT1608SURCK-AMT
- D40, D41, D42, D49: MOUSER PN 720-Q65113A5260 -> 720-Q65113A7469
Changed lines of the file:
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@@
 			)
 		)
-		(property "MOUSER PN" "720-Q65113A7467"
+		(property "MOUSER PN" "604-APT1608SURCK-AMT "
 			(at 342.9 36.83 0)
 			(hide yes)
@@
 			)
 		)
-		(property "MOUSER PN" "720-Q65113A5260"
+		(property "MOUSER PN" "720-Q65113A7469"
 			(at 375.92 54.61 0)
 			(hide yes)
@@
 			)
 		)
-		(property "MOUSER PN" "720-Q65113A7467"
+		(property "MOUSER PN" "604-APT1608SURCK-AMT "
 			(at 342.9 72.39 0)
 			(hide yes)
@@
 			)
 		)
-		(property "MOUSER PN" "720-Q65113A5260"
+		(property "MOUSER PN" "720-Q65113A7469"
 			(at 375.92 36.83 0)
 			(hide yes)
@@
 			)
 		)
-		(property "MOUSER PN" "720-Q65113A5260"
+		(property "MOUSER PN" "720-Q65113A7469"
 			(at 311.15 54.61 0)
 			(hide yes)
@@
 			)
 		)
-		(property "MOUSER PN" "720-Q65113A5260"
+		(property "MOUSER PN" "720-Q65113A7469"
 			(at 375.92 72.39 0)
 			(hide yes)
@@
 			)
 		)
-		(property "MOUSER PN" "720-Q65113A7467"
+		(property "MOUSER PN" "604-APT1608SURCK-AMT "
 			(at 342.9 54.61 0)
 			(hide yes)
