File: usb_interface.kicad_sch (KiCad schematic)
At the start: 10 parts, among them J4 USB_C_Receptacle_USB2.0_14P, U1 USBLC6-2SC6, U3 LD1117S33TR

Commit message: feat: added vias
Connections:
- net USB_D+: now also U1.4 (I/O2); no longer U1.3 (I/O2)
- net USB_D-: now also U1.6 (I/O1); no longer U1.1 (I/O1)
- net VBUS: now also J4.B5 (CC2), R18.2
- net at J4.A6 (D+), J4.B6 (D+): now also U1.3 (I/O2); no longer U1.4 (I/O2)
- net at J4.A7 (D-), J4.B7 (D-): now also U1.1 (I/O1); no longer U1.6 (I/O1)
Changed lines of the file:
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@@
+	)
+	(junction
+		(at 90.17 86.36)
+		(diameter 0)
+		(color 0 0 0 0)
 	)
 	(junction
@@
 	(wire
 		(pts
-			(xy 90.17 88.9) (xy 90.17 78.74)
+			(xy 90.17 88.9) (xy 90.17 86.36)
 		)
 		(stroke
@@
 	(wire
 		(pts
+			(xy 90.17 86.36) (xy 102.87 86.36)
+		)
+		(stroke
+			(width 0)
+			(type default)
+		)
+	)
+	(wire
+		(pts
 			(xy 90.17 78.74) (xy 81.28 78.74)
 		)
@@
 	(wire
 		(pts
-			(xy 81.28 86.36) (xy 102.87 86.36)
+			(xy 81.28 86.36) (xy 90.17 86.36)
 		)
 		(stroke
@@
 		(pts
 			(xy 92.71 83.82) (xy 81.28 83.82)
+		)
+		(stroke
+			(width 0)
+			(type default)
+		)
+	)
+	(wire
+		(pts
+			(xy 90.17 86.36) (xy 90.17 78.74)
 		)
 		(stroke
@@
 		(lib_id "Power_Protection:USBLC6-2SC6")
 		(at 90.17 93.98 0)
-		(mirror y)
 		(unit 1)
 		(body_style 1)
@@
 		(dnp no)
 		(property "Reference" "U1"
-			(at 89.154 101.092 0)
+			(at 91.186 101.092 0)
 			(show_name no)
 			(do_not_autoplace no)
@@
 		)
 		(property "Value" "USBLC6-2SC6"
-			(at 89.154 103.632 0)
+			(at 91.186 103.632 0)
 			(show_name no)
 			(do_not_autoplace no)
@@
 		)
 		(property "Footprint" "Package_TO_SOT_SMD:SOT-23-6"
-			(at 88.9 100.33 0)
+			(at 91.44 100.33 0)
 			(hide yes)
 			(show_name no)
@@
 		)
 		(property "Datasheet" "https://www.st.com/resource/en/datasheet/usblc6-2.pdf"
-			(at 88.9 102.235 0)
-			(hide yes)
-			(show_name no)
+			(at 91.44 102.235 0)
+			(hide yes)
+			(show_name no)

Commit message: feat: finished vias
Connections:
- net VBUS: no longer J4.B5 (CC2), R18.2
- new net: J4.B5 (CC2), R18.2
Changed lines of the file:
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@@
-	)
-	(junction
-		(at 90.17 86.36)
-		(diameter 0)
-		(color 0 0 0 0)
 	)
 	(junction
@@
 	(wire
 		(pts
-			(xy 90.17 88.9) (xy 90.17 86.36)
-		)
-		(stroke
-			(width 0)
-			(type default)
-		)
-	)
-	(wire
-		(pts
 			(xy 234.95 86.36) (xy 242.57 86.36)
 		)
@@
 	(wire
 		(pts
-			(xy 90.17 86.36) (xy 102.87 86.36)
+			(xy 81.28 86.36) (xy 102.87 86.36)
 		)
 		(stroke
@@
 	(wire
 		(pts
-			(xy 81.28 86.36) (xy 90.17 86.36)
-		)
-		(stroke
-			(width 0)
-			(type default)
-		)
-	)
-	(wire
-		(pts
 			(xy 191.77 86.36) (xy 195.58 86.36)
 		)
@@
 	(wire
 		(pts
-			(xy 90.17 86.36) (xy 90.17 78.74)
-		)
-		(stroke
+			(xy 90.17 78.74) (xy 90.17 88.9)
+		)
+		(stroke

Commit message: feat: started writing BOM
Parts:
- C17: LCSC Part # (none) -> C49678; MOUSER PN (none) -> 581-0805YC104M4T2A
- C18, C19: LCSC Part # (none) -> C15850; MOUSER PN (none) -> 581-KGM21AR71C106MU
- F1: LCSC Part # (none) -> C7542952; MOUSER PN (none) -> 576-1206L075SLYR
- FB1: LCSC Part # (none) -> C80165; MOUSER PN (none) -> 81-BLM18PG221SN1D
- J4: LCSC Part # (none) -> C319148; MOUSER PN (none) -> 640-USB4105-GF-A
- R17, R18: LCSC Part # (none) -> C14677; MOUSER PN (none) -> 603-RE0603FRE075K1L
- U1: LCSC Part # (none) -> C2827654; MOUSER PN (none) -> 511-USBLC6-2SC6
- U3: LCSC Part # (none) -> C86781; MOUSER PN (none) -> 511-LD1117S33

Commit message: feat: finished BOM
Parts:
- C18, C19: MOUSER PN 581-KGM21AR71C106MU -> 603-CC0805MKX77BB106
Changed lines of the file:
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@@
 			)
 		)
-		(property "MOUSER PN" "581-KGM21AR71C106MU"
+		(property "MOUSER PN" "603-CC0805MKX77BB106"
 			(at 195.58 96.52 0)
 			(hide yes)
@@
 			)
 		)
-		(property "MOUSER PN" "581-KGM21AR71C106MU"
-			(at 242.57 96.52 0)
-			(hide yes)
+		(property "MOUSER PN" "603-CC0805MKX77BB106"
+			(at 242.57 96.52 0)
+			(hide yes)
