File: CAN-serializer.kicad_pcb (KiCad board)
At the start: 4 copper layers, 68.8 x 39.5 mm, 111 parts, among them J2 SPI connector, J3 I2C connector, J4 USB_C_Receptacle_USB2.0_14P, J5 CAN interfaces, J6 USART2 connector, J7 Debug, SW1 SW_DIP_x03, SW2 RESET, U1 USBLC6-2SC6, U13 MCP2562FD, U14 MCP2562FD, U15 MCP2562FD, U2 STM32G473CCTx, U3 LD1117S33TR, Y2 16MHz

Commit message: feat: added vias
Parts:
- removed D36: GREEN LED, LED_SMD:LED_0603_1608Metric_Pad1.05x0.95mm_HandSolder
- removed R8: 680R, Resistor_SMD:R_0603_1608Metric_Pad0.98x0.95mm_HandSolder
- moved D24 11.8 mm to (189.8, 63.8)
- moved D26 11.7 mm to (189.3, 66.2)
- moved D30 11.2 mm to (201.3, 66.2)
- moved D28 11.2 mm to (201.8, 63.8)
- moved D29 8.75 mm to (193.8, 63.8)
- moved D31 8.69 mm to (193.2, 66.2)
- moved D33 7.69 mm to (181.8, 63.7)
- moved D35 7.69 mm to (181.2, 66.2)
- moved D32 6.20 mm to (185.8, 63.8)
- moved D34 6.19 mm to (185.2, 66.2)
- moved C17 3.15 mm to (175.5, 43.5)
- moved C18 2.87 mm to (175.5, 46.5)
- moved C11 2.07 mm to (175.3, 58.4)
- moved C9 2.07 mm to (175.3, 52.4)
- moved Y2 2.07 mm to (175.3, 55.4)
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Connections:
- J4 pad B5: Net-(J4-CC2) -> /USB interface/VBUS
- R18 pad 2: Net-(J4-CC2) -> /USB interface/VBUS
- U1 pad 1: /MCU/USB_D- -> Net-(J4-D--PadA7)
- U1 pad 3: /MCU/USB_D+ -> Net-(J4-D+-PadA6)
- U1 pad 4: Net-(J4-D+-PadA6) -> /MCU/USB_D+
- U1 pad 6: Net-(J4-D--PadA7) -> /MCU/USB_D-
- U2 pad 2: /MCU/CAN3_LED_RX -> /MCU/CAN1_LED_RX
- U2 pad 4: /MCU/CAN1_LED_RX -> /MCU/CAN2_LED_RX
- U2 pad 8: /MCU/CAN2_LED_RX -> /MCU/CAN2_LED_TX
- U2 pad 9: /MCU/CAN2_LED_TX -> /MCU/CAN3_LED_RX
Routing:
- net /CAN interfaces/CAN_H1: track 0.00 -> 41.0 mm, vias 0 -> 2
- net +3V3: track 0.00 -> 40.5 mm, vias 0 -> 12
- net /CAN interfaces/CAN_L1: track 0.00 -> 40.1 mm, vias 0 -> 2
- net /CAN interfaces/CAN_L2: track 0.00 -> 33.8 mm, vias 0 -> 2
- net /CAN interfaces/CAN_H2: track 0.00 -> 29.1 mm, vias 0 -> 2
- net /CAN interfaces/CAN_L3: track 0.00 -> 28.3 mm, vias 0 -> 2
- net /MCU/CAN3_LED_TX: track 0.00 -> 27.5 mm, vias 0 -> 2
- net /MCU/SWO: track 0.00 -> 26.9 mm
- net +5V: track 0.00 -> 26.5 mm, vias 0 -> 3
- net /MCU/USART2_TX: track 0.00 -> 23.5 mm
- net /MCU/SPI_CS: track 0.00 -> 22.0 mm
- net /MCU/USART2_RX: track 0.00 -> 21.8 mm
- net /MCU/SWDIO: track 0.00 -> 21.1 mm
- net /MCU/SWCLK: track 0.00 -> 19.7 mm
- net /MCU/SPI_MOSI: track 0.00 -> 18.6 mm
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- added copper zone on B.Cu, net GND
- added copper zone on F.Cu, net GND
- added copper zone on In1.Cu, net GND
- added copper zone on In2.Cu, net GND

Commit message: feat: finished vias
Parts:
- added H1: MountingHole, MountingHole:MountingHole_2.2mm_M2_ISO14580, F.Cu at (143.8, 74.0)
- added H2: MountingHole, MountingHole:MountingHole_2.2mm_M2_ISO14580, F.Cu at (172.0, 71.2)
- moved J4 1.50 mm to (204.8, 55.2)
- moved C12 1.19 mm to (191.2, 50.0)
- moved D43 1.19 mm to (204.6, 45.8)
- moved D45 1.19 mm to (199.5, 45.8)
- moved J3 1.19 mm to (196.0, 41.8)
- moved R1 1.19 mm to (204.6, 47.2)
- moved R2 1.19 mm to (201.0, 47.2)
- moved R3 1.19 mm to (201.0, 44.2)
- moved R4 1.19 mm to (204.6, 44.2)
- moved C20 0.25 mm to (165.5, 66.8)
- moved SW2 0.25 mm to (205.2, 69.0)
Connections:
- J4 pad B5: /USB interface/VBUS -> Net-(J4-CC2)
- R18 pad 2: /USB interface/VBUS -> Net-(J4-CC2)
Routing:
- net GND: track 13.4 -> 90.0 mm, vias 4 -> 48
- net /MCU/RESET: track 13.6 -> 89.4 mm, vias 0 -> 3
- net +5V: track 26.5 -> 60.0 mm, vias 3 -> 4
- net /USB interface/VBUS: track 0.00 -> 30.8 mm, vias 0 -> 4
- net /CAN interfaces/CAN3_TX: track 0.00 -> 29.8 mm, vias 0 -> 2
- net /MCU/CAN1_LED_RX: track 0.00 -> 29.6 mm, vias 0 -> 2
- net /MCU/SWDIO: track 21.1 -> 48.9 mm, vias 0 -> 2
- net +3V3: track 40.5 -> 68.2 mm, vias 12 -> 21
- net /CAN interfaces/CAN3_RX: track 0.00 -> 25.7 mm, vias 0 -> 2
- net /CAN interfaces/CAN2_RX: track 0.00 -> 24.0 mm, vias 0 -> 2
- net /MCU/SWO: track 26.9 -> 49.2 mm, vias 0 -> 2
- net /MCU/I2C_SCL: track 0.00 -> 22.3 mm
- net /MCU/SWCLK: track 19.7 -> 41.9 mm, vias 0 -> 2
- net /MCU/I2C_SDA: track 0.00 -> 21.4 mm
- net /CAN interfaces/CAN1_RX: track 0.00 -> 21.0 mm, vias 0 -> 2
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- added copper zone on In2.Cu, net +3V3
Other:
- board size 68.8 x 39.5 mm -> 68.1 x 39.5 mm

Commit message: feat: finished first prototype
Parts:
- added G***: LOGO, Eagle_Logos:newlogo, B.Cu at (155.2, 72.0)
- added G***: LOGO, Eagle_Logos:logo_12mm3_3000scale, B.Cu at (194.2, 49.2)
Other:
- board text added: "3V3"
- board text added: "@ale-giustina RP-MBD 13/10/2026 Rev 1.0.0"
- board text added: "CAN-serializer"
- board text added: "CAN1+"
- board text added: "CAN1-"
- board text added: "CAN2+"
- board text added: "CAN2-"
- board text added: "CAN3+"
- board text added: "CAN3-"
- board text added: "CS"
- board text added: "Che Guevara tits"
- board text added: "GND"
- board text added: "MIO"
- board text added: "MOI"
- board text added: "ON ->"
- board text added: "Perché se vuoi che hardware faccia qualcosa, devi imparare a farlo tu"
- board text added: "SCK"
- board text added: "SCL"
- board text added: "SDA"
- board text added: "USB"

Commit message: feat: started writing BOM
Parts:
- removed the G*** at (194.2, 49.2)
- removed SW1: SW_DIP_x03, Button_Switch_SMD:SW_DIP_SPSTx03_Slide_6.7x9.18mm_W6.73mm_P2.54mm_LowProfile_JPin
- added J1: Conn_01x02, Connector_PinHeader_2.00mm:PinHeader_1x02_P2.00mm_Vertical, F.Cu at (156.2, 75.5)
- added J8: Conn_01x02, Connector_PinHeader_2.00mm:PinHeader_1x02_P2.00mm_Vertical, F.Cu at (156.2, 72.5)
- added J9: Conn_01x02, Connector_PinHeader_2.00mm:PinHeader_1x02_P2.00mm_Vertical, F.Cu at (156.2, 69.5)
- moved H2 27.4 mm to (197.0, 60.0)
- moved C10 3.50 mm to (202.0, 61.8), turned to 180 degrees
- moved R21 2.31 mm to (151.0, 69.5)
- moved R20 2.08 mm to (151.0, 72.5)
- moved R19 1.96 mm to (151.0, 75.5)
- moved SW2 1.82 mm to (205.8, 67.2)
- moved H1 1.41 mm to (144.8, 73.0)
- moved C47 1.17 mm to (171.3, 62.2)
- moved R49 0.83 mm to (169.6, 60.3)
- moved C46 0.75 mm to (171.3, 53.0)
- moved R18 0.75 mm to (194.5, 49.0)
- moved R44 0.58 mm to (169.6, 45.7)
- moved R14 0.50 mm to (169.6, 58.5)
- moved R47 0.42 mm to (169.6, 51.2)
- moved C45 0.33 mm to (171.3, 43.8)
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Connections:
- R19 pad 2: /CAN interfaces/CAN_L3 -> /CAN interfaces/CAN_L1
- R21 pad 2: /CAN interfaces/CAN_L1 -> /CAN interfaces/CAN_L3
Routing:
- net GND: track 90.0 -> 106.1 mm, vias 48 -> 59
- net /CAN interfaces/CAN_L3: track 28.3 -> 21.2 mm
- net /MCU/SWDIO: track 48.9 -> 52.3 mm
- net /CAN interfaces/CAN_L1: track 40.1 -> 43.3 mm
- net /CAN interfaces/CAN_H3: track 17.0 -> 14.2 mm
- net /MCU/SWCLK: track 41.9 -> 44.6 mm
- net /CAN interfaces/CAN_L2: track 33.8 -> 31.5 mm
- net +5V: track 60.0 -> 62.2 mm
- net /MCU/I2C_SCL: track 22.3 -> 21.0 mm, vias 0 -> 2
- net /CAN interfaces/CAN_H1: track 41.0 -> 39.8 mm
- net /MCU/I2C_SDA: track 21.4 -> 20.3 mm
- net /CAN interfaces/CAN_H2: track 29.1 -> 28.0 mm
- net /MCU/CAN3_LED_RX: track 15.2 -> 14.4 mm
- net Net-(J4-CC2): track 7.47 -> 8.07 mm
- net /MCU/CAN1_LED_RX: track 29.6 -> 29.0 mm
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Other:
- board text added: "RX"
- board text added: "TX"
- board text removed: "Che Guevara tits"
- board text removed: "ON ->"

Commit message: feat: finished BOM
Parts:
- added G***: LOGO, Eagle_Logos:logo_10mm3_3500scale, B.Cu at (194.0, 49.0)

Commit message: feat: first batch
Parts:
- removed the G*** at (194.0, 49.0)
- added G***: LOGO, MIALIBRERIA:LOGO, B.Cu at (151.1, 50.6)
- moved G*** 40.8 mm to (196.0, 71.0)
Routing:
- net /USB interface/VBUS: track 30.8 -> 31.7 mm
- net /MCU/RESET: track 89.3 -> 88.4 mm
- net GND: vias 59 -> 61
Other:
- board text added: "Il CAN è come le cipolle... Puzza? Sì... no! Ah, ti fa piangere? No! Ah, lo lasci al sole diventa marrone e poi spuntano i peletti bianchi? No! Strati! Il CAN ha gli strati, le cipolle hanno gli strati! Capite? Tutti e due hanno gli strati!"
- board text added: "\(°□°)/"
